File: pcb/geodude-carrier/geodude-carrier.kicad_sch (KiCad schematic)
At the start: 32 parts

Commit message: Fix carrier PCB schematic: 5 power rails, PCA9685 on 3.3V
- +12V (servo power, ESC, fan)
- +7V4 (elbow servo power)
- +5V_SERVO (wrist servo power, from buck 3)
- +5V_LOGIC (from Pi 5V, general purpose)
- +3V3 (from Pi 3.3V, PCA9685 VCC, I2C bus)
Parts:
- added J_3V3: 3V3_Input, symbol Connector:Screw_Terminal_01x02
- added J_5V_LOGIC: 5V_Logic_Input, symbol Connector:Screw_Terminal_01x02
- J_5V_SERVO: renamed from J_5V; value 5V_Input -> 5V_Servo_Input
Connections:
- net +12V: now also J_3V3.1 (Pin_1), J_5V_LOGIC.1 (Pin_1)
Other:
- note added: "1. PCA9685 VCC = 3.3V (from Pi 3.3V pin)"
- note added: "10. I2C breakout ports powered by +3V3 rail"
- note added: "5-Rail Power Distribution + Servo/ESC/Fan Control via PCA9685"
- note added: "6. 5V_SERVO wrist servos (SV4,SV5,SV9,SV10) fused at 3A (from buck converter 3)"
- note added: "9. 5 power rails: +12V (battery), +7V4 (buck1), +5V_SERVO (buck3), +5V_LOGIC (Pi 5V), +3V3 (Pi 3.3V)"
- note removed: "1. PCA9685 VCC = 5V logic supply"
- note removed: "6. 5V servos (SV4,SV5,SV9,SV10) fused at 3A"
- note removed: "Power Distribution + Servo/ESC/Fan Control via PCA9685"
